File: penrosekite.kicad_pcb (KiCad board)
At the start: 2 copper layers, 50 x 47.5 mm, 21 parts, among them J1 Conn_01x03_Female, J2 Conn_01x03_Female, J3 Conn_01x03_Male, J4 Conn_01x03_Male, M2.1 MountingHole_2.1mm, SW1 SW_DPDT_x2

Commit message: shifted ports  on penrose rhombi to enforce all matching rules. fixed flipped ports on penrose dart.
going to make new gerbers later.
Other:
- board text added: "GND VCC DATA"

Commit message: increased mounting hole size to M3
increased mounting hole size to M3 to accomidate plastic adhesive mounting hole standoffs. makes the silkscreen a bit cramped and the VCC   route a bit long, but maybe I will make the top pour VCC instead of ground later idk.
Parts:
- removed M2.1 (x2): MountingHole_2.1mm, MountingHole:MountingHole_2.1mm
- added M3: MountingHole_3.2mm_M3_ISO7380, MountingHole:MountingHole_3.2mm_M3_ISO7380, F.Cu at (140.5, 97.2)
- added M3: MountingHole_3.2mm_M3_ISO7380, MountingHole:MountingHole_3.2mm_M3_ISO7380, F.Cu at (117.0, 114.3)
- added M3: MountingHole_3.2mm_M3_ISO7380, MountingHole:MountingHole_3.2mm_M3_ISO7380, F.Cu at (138.4, 117.8)
- M3: renamed from M2.1; value MountingHole_2.1mm -> MountingHole_3.2mm_M3_ISO7380; footprint MountingHole:MountingHole_2.1mm -> MountingHole:MountingHole_3.2mm_M3_ISO7380
- moved M3 0.16 mm to (120.3, 92.8)

Commit message: minor tweaks and diagrams
Tweaks to silkscreen and stuff also added a diagram to explain switch on board. Also made top layer VCC on penrose kite.
Parts:
- turned C3 to 18 degrees
Routing:
- net VCC: track 114.3 -> 102.5 mm
- net GND: track 21.7 -> 33.2 mm, vias 11 -> 8
- added copper zone on F.Cu, net VCC
- removed copper zone on F.Cu, net GND
Other:
- board text added: "α"
- board text added: "β"
Changed lines of the file:
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@@
   (general
     (thickness 1.6)
-    (drawings 84)
-    (tracks 86)
+    (drawings 86)
+    (tracks 84)
     (zones 0)
     (modules 22)
@@
     (uvia_dia 0.3)
     (uvia_drill 0.1)
-    (add_net GND)
     (add_net "Net-(D1-Pad2)")
     (add_net "Net-(D1-Pad4)")
@@
     (uvia_dia 0.3)
     (uvia_drill 0.1)
+    (add_net GND)
     (add_net VCC)
   )
@@
   )
   (module Capacitor_SMD:C_0805_2012Metric_Pad1.18x1.45mm_HandSolder (layer F.Cu)
-    (at 141.9225 103.6955 198)
+    (at 141.9225 103.6955 18)
     (descr "Capacitor SMD 0805 (2012 Metric), square (rectangular) end terminal, IPC_7351 nominal with elongated pad for handsoldering. (Body size source: IPC-SM-782 page 76, https://www.pcb-3d.com/wordpress/wp-content/uploads/ipc-sm-782a_amendment_1_and_2.pdf, https://docs.google.com/spreadsheets/d/1BsfQQcO9C6DZCsRaXUlFlo91Tg2WpOkGARC1WS5S8t0/edit?usp=sharing), generated with kicad-footprint-generator")
     (tags "capacitor handsolder")
@@
       (effects (font (size 0.5 0.5) (thickness 0.08)))
     )
-    (pad 2 smd roundrect (at 1.0375 0 198) (size 1.175 1.45) (layers F.Cu F.Paste F.Mask) (roundrect_rratio 0.2127659574468085)
-      (net 1 VCC))
-    (pad 1 smd roundrect (at -1.0375 0 198) (size 1.175 1.45) (layers F.Cu F.Paste F.Mask) (roundrect_rratio 0.2127659574468085)
+    (pad 2 smd roundrect (at 1.0375 0 18) (size 1.175 1.45) (layers F.Cu F.Paste F.Mask) (roundrect_rratio 0.2127659574468085)
+      (net 1 VCC))
+    (pad 1 smd roundrect (at -1.0375 0 18) (size 1.175 1.45) (layers F.Cu F.Paste F.Mask) (roundrect_rratio 0.2127659574468085)
       (net 2 GND))
     (model ${KISYS3DMOD}/Capacitor_SMD.3dshapes/C_0805_2012Metric.wrl
@@
     (at 129.794 104.394 306)
     (descr "MSS22D18 MINI Miniature SMD SMT Slide Switch 2P2T ")
-    (fp_text reference SW1 (at 0.5 -5.5 126) (layer F.SilkS)
+    (fp_text reference SW1 (at 0.239373 -1.634503 216) (layer F.SilkS)
       (effects (font (size 1 1) (thickness 0.15)))
     )
@@
       (rotate (xyz -90 0 90))
     )
+  )
+  (gr_text α (at 134.28472 101.1682 306) (layer F.SilkS)
+    (effects (font (size 1 1) (thickness 0.15)))
+  )
+  (gr_text β (at 125.10516 107.86364 126) (layer F.SilkS)
+    (effects (font (size 1 1) (thickness 0.15)))
   )
   (gr_text "GND\nVCC\nDATA" (at 143.2306 108.0262 198) (layer B.SilkS)
@@
   (segment (start 128.7145 91.313) (end 127.222789 90.137711) (width 1) (layer F.Cu) (net 1))
   (segment (start 125.838639 91.040639) (end 127.222789 90.137711) (width 1) (layer F.Cu) (net 1))
-  (segment (start 142.842147 105.682902) (end 140.935779 104.016105) (width 1) (layer F.Cu) (net 1))
   (segment (start 116.946961 105.620017) (end 117.572721 108.143605) (width 1) (layer F.Cu) (net 1))
   (segment (start 127.324584 120.563941) (end 128.905 118.364) (width 1) (layer F.Cu) (net 1))
@@
   (segment (start 128.905 118.364) (end 130.786533 118.404033) (width 1) (layer F.Cu) (net 1))
   (segment (start 131.949031 117.534531) (end 132.08 115.57) (width 1) (layer F.Cu) (net 1))
-  (segment (start 140.935779 104.016105) (end 138.900359 102.082141) (width 1) (layer F.Cu) (net 1))
-  (segment (start 143.764 101.727) (end 144.411014 103.707514) (width 1) (layer F.Cu) (net 1))
-  (segment (start 144.411014 103.707514) (end 144.757677 105.305323) (width 1) (layer F.Cu) (net 1))
-  (segment (start 146.926026 106.724544) (end 144.757677 105.305323) (width 1) (layer F.Cu) (net 1))
-  (segment (start 142.842147 105.682902) (end 138.6713 110.5408) (width 1) (layer F.Cu) (net 1))
   (segment (start 132.08 115.57) (end 138.6713 110.5408) (width 1) (layer F.Cu) (net 1))
   (segment (start 113.8555 108.458) (end 117.348 109.601) (width 1) (layer F.Cu) (net 1))
@@
   (segment (start 114.681 106.1085) (end 115.128835 104.898665) (width 1) (layer F.Cu) (net 1))
   (segment (start 114.185846 102.497282) (end 115.128835 104.898665) (width 1) (layer F.Cu) (net 1))
-  (segment (start 138.900359 102.082141) (end 135.579082 98.926418) (width 1) (layer F.Cu) (net 1))
-  (segment (start 135.579082 98.926418) (end 134.178936 97.596064) (width 1) (layer F.Cu) (net 1))
-  (segment (start 134.178936 97.596064) (end 132.994173 96.470355) (width 1) (layer F.Cu) (net 1))
   (segment (start 133.402689 88.130443) (end 130.285771 93.551729) (width 1) (layer F.Cu) (net 1))
   (segment (start 130.285771 93.551729) (end 131.251571 94.927789) (width 1) (layer F.Cu) (net 1))
@@
   (segment (start 113.792 106.426) (end 113.157 108.204) (width 1) (layer F.Cu) (net 1))
   (segment (start 113.157 108.204) (end 113.8555 108.458) (width 1) (layer F.Cu) (net 1))
-  (segment (start 140.935779 104.016105) (end 141.791142 101.871058) (width 1) (layer F.Cu) (net 1))
-  (segment (start 143.764 101.727) (end 141.791142 101.871058) (width 1) (layer F.Cu) (net 1))
   (segment (start 123.302494 99.909094) (end 125.838639 91.040639) (width 1) (layer F.Cu) (net 1))
   (segment (start 122.448159 103.357841) (end 123.302494 99.909094) (width 1) (layer F.Cu) (net 1))
   (segment (start 116.946961 105.620017) (end 122.448159 103.357841) (width 1) (layer F.Cu) (net 1))
+  (segment (start 142.842147 105.682902) (end 142.909221 103.374895) (width 1) (layer F.Cu) (net 1))
+  (segment (start 142.909221 103.374895) (end 132.994173 96.470355) (width 1) (layer F.Cu) (net 1))
+  (segment (start 142.842147 105.682902) (end 146.926026 106.724544) (width 1) (layer F.Cu) (net 1))
   (segment (start 115.599279 107.502395) (end 116.205 103.886) (width 0.25) (layer F.Cu) (net 2))
-  (segment (start 116.205 103.886) (end 121.504525 101.948695) (width 0.25) (layer F.Cu) (net 2))
   (via (at 114.6175 107.442) (size 0.8) (drill 0.4) (layers F.Cu B.Cu) (net 2))
   (segment (start 115.599279 107.502395) (end 114.6175 107.442) (width 0.25) (layer F.Cu) (net 2))
-  (via (at 120.2055 101.473) (size 0.8) (drill 0.4) (layers F.Cu B.Cu) (net 2))
   (via (at 124.587 115.5065) (size 0.8) (drill 0.4) (layers F.Cu B.Cu) (net 2))
   (via (at 128.4605 116.967) (size 0.8) (drill 0.4) (layers F.Cu B.Cu) (net 2))
-  (via (at 141.478 109.474) (size 0.8) (drill 0.4) (layers F.Cu B.Cu) (net 2))
-  (segment (start 141.478 109.474) (end 144.272 106.6165) (width 0.25) (layer F.Cu) (net 2))
   (via (at 130.429 90.424) (size 0.8) (drill 0.4) (layers F.Cu B.Cu) (net 2))
   (via (at 132.715 93.853) (size 0.8) (drill 0.4) (layers F.Cu B.Cu) (net 2))
-  (via (at 143.383 104.267) (size 0.8) (drill 0.4) (layers F.Cu B.Cu) (net 2))
-  (segment (start 142.909221 103.374895) (end 143.383 104.267) (width 0.25) (layer F.Cu) (net 2))
-  (segment (start 143.383 104.267) (end 144.2466 106.3498) (width 0.25) (layer F.Cu) (net 2))
-  (segment (start 144.2466 106.3498) (end 141.478 109.474) (width 0.25) (layer F.Cu) (net 2))
-  (via (at 125.222 108.9152) (size 0.8) (drill 0.4) (layers F.Cu B.Cu) (net 2))
-  (via (at 134.2136 100.6856) (size 0.8) (drill 0.4) (layers F.Cu B.Cu) (net 2))
-  (via (at 136.4742 108.2548) (size 0.8) (drill 0.4) (layers F.Cu B.Cu) (net 2))
+  (segment (start 131.347786 86.637468) (end 129.168301 89.458787) (width 1) (layer F.Cu) (net 2))
+  (segment (start 129.168301 89.458787) (end 130.429 90.424) (width 1) (layer F.Cu) (net 2))
+  (segment (start 132.715 93.853) (end 134.213827 94.791645) (width 1) (layer F.Cu) (net 2))
+  (via (at 140.92428 110.23092) (size 0.8) (drill 0.4) (layers F.Cu B.Cu) (net 2))
+  (segment (start 122.936 115.8455) (end 124.587 115.5065) (width 1) (layer F.Cu) (net 2))
+  (segment (start 124.587 115.5065) (end 127.09144 115.94084) (width 1) (layer F.Cu) (net 2))
+  (segment (start 127.09144 115.94084) (end 128.4605 116.967) (width 1) (layer F.Cu) (net 2))
+  (segment (start 128.4605 116.967) (end 130.109486 116.972169) (width 1) (layer F.Cu) (net 2))
+  (segment (start 140.92428 110.23092) (end 141.312949 111.331934) (width 1) (layer F.Cu) (net 2))
+  (segment (start 140.92428 110.23092) (end 141.4018 105.65892) (width 1) (layer F.Cu) (net 2))
+  (segment (start 141.4018 105.65892) (end 141.29403 105.27901) (width 1) (layer F.Cu) (net 2))
+  (segment (start 141.29403 105.27901) (end 140.935779 104.016105) (width 1) (layer F.Cu) (net 2))
+  (via (at 141.29403 105.27901) (size 0.8) (drill 0.4) (layers F.Cu B.Cu) (net 2))
+  (via (at 120.41613 102.34657) (size 0.8) (drill 0.4) (layers F.Cu B.Cu) (net 2))
+  (segment (start 121.504525 101.948695) (end 120.41613 102.34657) (width 1) (layer F.Cu) (net 2))
+  (segment (start 116.205 103.886) (end 120.41613 102.34657) (width 0.25) (layer F.Cu) (net 2))
+  (segment (start 115.599279 107.502395) (end 114.693672 107.469204) (width 1) (layer F.Cu) (net 2))
   (segment (start 127.287388 92.047641) (end 125.73 98.7425) (width 0.25) (layer F.Cu) (net 3))
   (segment (start 125.73 98.7425) (end 126.365 99.949) (width 0.25) (layer F.Cu) (net 3))
@@
   (segment (start 126.110964 103.57799) (end 125.313278 100.713121) (width 0.25) (layer F.Cu) (net 10))
   (segment (start 126.110964 103.57799) (end 133.477036 105.21001) (width 0.25) (layer F.Cu) (net 10))
-  (zone (net 2) (net_name GND) (layer F.Cu) (hatch edge 0.508)
+  (zone (net 1) (net_name VCC) (layer F.Cu) (hatch edge 0.508)
     (connect_pads (clearance 0.508))
     (min_thickness 0.254)
